File: Tornado.kicad_pcb (KiCad board)
At the start: 4 copper layers, 22.9 x 22.9 mm, 42 parts, among them J1 MOLEX, SW1 ID, U1 AP63205WU, U2 STM32G431KBUx, U3 LSM6DS3, U4 AP2112K-3.3, U5 TCAN1057A, Y1 32MHz

Commit message: Added graphics
Parts:
- moved C20 0.25 mm to (149.7, 89.8)
Routing:
- net +5V: track 49.6 -> 52.3 mm, vias 5 -> 4
- net /SCL: track 24.6 -> 22.1 mm
- net /DOUT: track 26.1 -> 24.0 mm
- net GND: track 86.0 -> 87.7 mm, vias 21 -> 19
- net /SDA: track 25.5 -> 27.1 mm, vias 2 -> 3
- net /RGB: track 12.3 -> 11.2 mm
- net +3.3V: track 69.6 -> 68.7 mm
- net /PWR_LED: track 27.3 -> 27.9 mm
- net /IMU_INT: track 6.32 -> 5.87 mm, vias 2 -> 0
